File: froggy_hw/froggy_hw.kicad_sch (KiCad schematic)
At the start: 42 parts, among them J1 I2C, J2 SWD, P1 TC2030_STM32, SW1 SW_Push, U1 STM32F030F4Px, U2 SN75176AD, U3 TLP2361, U4 TLP2361, U5 TLP2361, U6 B0505S-1WR3

Commit message: moved to esp32
Parts:
- removed C28 (x6): 100n, otter:C_0402, symbol Device:C_Small
- removed C28: DNP, otter:C_0402, symbol Device:C_Small
- removed C29 (x3): 4u7, otter:C_0805, symbol Device:C_Small
- removed D4: 12V, otter:LED_0603_1608Metric, symbol Device:LED
- removed J2: SWD, otter:PinSocket_1x04_P2.54mm_Vertical_center, symbol Connector_Generic:Conn_01x04
- removed L1: 4u7, Inductor_SMD:L_1210_3225Metric, symbol Device:L_Small
- removed P1: TC2030_STM32, otter:TC2030, symbol otter:TC2030-CTX-Tag-Connect
- removed R12, R9: 200, otter:R_0402, symbol Device:R_Small
- removed R2: 580, otter:R_0805, symbol Device:R_Small
- removed R26: 13k, otter:R_0402, symbol Device:R_Small
- removed R27: 5k1, otter:R_0402, symbol Device:R_Small
- removed U1: STM32F030F4Px, Package_SO:TSSOP-20_4.4x6.5mm_P0.65mm, symbol MCU_ST_STM32F0:STM32F030F4Px
- removed U2: SN75176AD, Package_SO:SOIC-8_3.9x4.9mm_P1.27mm, symbol Interface_UART:SN75176AD
- removed U3, U4, U5: TLP2361, otter:TLP2361, symbol otter:TLP2361
- removed U6: B0505S-1WR3, otter:B0303S-1WR3, symbol otter:B0303S-1WR3
- added C11: 4u7, otter:C_0805, symbol Device:C_Small
- added D19: HEAT, otter:LED_0603_1608Metric, symbol Device:LED
- added D20: ERR, otter:LED_0603_1608Metric, symbol Device:LED
- added D6: OK, otter:LED_0603_1608Metric, symbol Device:LED
- added P2: TC2030-CTX-Tag-Connect-ESP32, otter:TC2030, symbol otter:TC2030-CTX-Tag-Connect-ESP32
- added R19, R7: 5k1, otter:R_0402, symbol Device:R_Small
- added SW2: SW_Push, Button_Switch_SMD:SW_SPST_EVQP7C, symbol Switch:SW_Push
- added U1: PCA9536DP, Package_SO:TSSOP-8_3x3mm_P0.65mm, symbol Interface_Expansion:PCA9536DP
- added U11: ESP32-C3-MINI-1, otter:ESP32-C3-MINI-1, symbol otter:ESP32-C3-MINI-1
- D4: value 12V -> 24V
- J1: footprint otter:PinSocket_1x04_P2.54mm_Vertical_center -> Connector_PinHeader_2.54mm:PinHeader_1x04_P2.54mm_Vertical_SMD_Pin1Left
- R1, R5: value 200 -> 22k
- R26: value 5k1 -> 22k
- R26: value 22k -> 100k
- R3: value 133 -> 22k; footprint otter:R_0805 -> otter:R_0402
- R4: value 580 -> 22k; footprint otter:R_0805 -> otter:R_0402
- R8: value 200 -> 5k1
Connections:
- net RS485_TX is gone; now on net +3V3: R8.2
- net +3V3: now also C1.1, J1.2 (Pin_2), C11.2, R19.1, R7.2, U1.8 (VDD), U11.3 (3V3); no longer J1.3 (Pin_3)
- net GND: now also J1.1 (Pin_1), C11.1, D19.1 (K), D20.1 (K), D6.1 (K), P2.5 (GND), SW2.2, U1.4 (VSS), U11.1 (GND), U11.11 (GND), U11.14 (GND), U11.2 (GND), U11.36 (GND), U11.37 (GND), U11.38 (GND), U11.39 (GND), U11.40 (GND), U11.41 (GND), U11.42 (GND), U11.43 (GND), U11.44 (GND), U11.45 (GND), U11.46 (GND), U11.47 (GND), U11.48 (GND), U11.49 (GND), U11.50 (GND), U11.51 (GND), U11.52 (GND), U11.53 (GND); no longer J1.4 (Pin_4), R1.1
- net IO: now also R8.1, SW2.1, U11.21 (IO7); no longer SW1.1
- net LED_0: now also U11.22 (IO8)
- net NOZZLE: now also U11.13 (IO1)
- net NTC: now also U11.5 (IO2)
- net RS485_DE: now also U11.16 (IO10)
- net SCL: now also J1.3 (Pin_3), U1.6 (SCL), U11.18 (IO4); no longer J1.2 (Pin_2)
- net SDA: now also J1.4 (Pin_4), U1.7 (SDA), U11.19 (IO5); no longer J1.1 (Pin_1)
- net VALVE: now also U11.12 (IO0)
- net at R5.1: now also U1.5 (IO3)
- net at R5.2: now also D5.2 (A)
- net at R1.2: now also D6.2 (A)
- net RS485_A: no longer names the net of R3.1
- net RS485_A: now also U1.2 (IO1); no longer R4.2
- net RS485_B: no longer names the net of R3.2
- net RS485_B: now also D19.2 (A)
- net RS485_GND: no longer names the net of R4.1
- net RS485_GND: now also U1.3 (IO2)
- new net: D20.2 (A), R4.2
- new net: R7.1, SW1.1, U11.20 (IO6)
- new net: R1.1, U1.1 (IO0)
- new net ESP32_EN: P2.6 (EN), R19.2, U11.8 (EN)
- new net ESP32_IO9: P2.2 (IO0), U11.23 (IO9)
- new net ESP32_RXD: P2.4 (RXD), U11.30 (RXD)
- new net ESP32_TXD: P2.3 (TXD), U11.31 (TXD)
- new net FAN: U11.6 (IO3)
- new net USB_D+: U11.27 (IO19)
- new net USB_D-: U11.26 (IO18)
- no-connect marks 2 -> 0
Other:
- sheet Out ports: added FAN; removed FAN_1, FAN_2, LED_1
- sheet Power & IO ports: added RS485_DE, RS485_RX, RS485_TX, USB_D+, USB_D-; removed RS485_A, RS485_B, RS485_GND
- note added: "PWM Fan Control"
- note added: "Program"
- note removed: "PWM Optional Fans"
- note removed: "SWD"
- moved on the sheet: D4, J1, R26, R27

Commit message: updated to new kicad version
Parts:
- renumbered D4 to D1, D4 to D3, R26 to R10, R26 to R11, R27 to R14, R27 to R15, R26 to R6
Changed lines of the file:
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@@
 (kicad_sch
-	(version 20231120)
+	(version 20250114)
 	(generator "eeschema")
-	(generator_version "8.0")
+	(generator_version "9.0")
 	(paper "A4")
+	(text "External IO\n"
+		(exclude_from_sim no)
+		(at 144.78 168.91 0)
+		(effects
+			(font
+				(size 1.27 1.27)
+				(color 255 153 0 1)
+			)
+			(justify left bottom)
+		)
+	)
+	(text "SK6812\n"
+		(exclude_from_sim no)
+		(at 101.0525 171.5295 0)
+		(effects
+			(font
+				(size 1.27 1.27)
+				(color 255 153 0 1)
+			)
+			(justify left bottom)
+		)
+	)
+	(text "PWM Fan Control"
+		(exclude_from_sim no)
+		(at 99.06 158.75 0)
+		(effects
+			(font
+				(size 1.27 1.27)
+				(color 255 153 0 1)
+			)
+			(justify left bottom)
+		)
+	)
+	(text "PWM Valve Control"
+		(exclude_from_sim no)
+		(at 102.87 151.13 0)
+		(effects
+			(font
+				(size 1.27 1.27)
+				(color 255 153 0 1)
+			)
+			(justify left bottom)
+		)
+	)
+	(text "DMX512\n"
+		(exclude_from_sim no)
+		(at 105.9575 176.4505 0)
+		(effects
+			(font
+				(size 1.27 1.27)
+				(color 255 153 0 1)
+			)
+			(justify left bottom)
+		)
+	)
+	(text "PWM Heater"
+		(exclude_from_sim no)
+		(at 101.6 153.67 0)
+		(effects
+			(font
+				(size 1.27 1.27)
+				(color 255 153 0 1)
+			)
+			(justify left bottom)
+		)
+	)
+	(text "Temperature Sensor\n"
+		(exclude_from_sim no)
+		(at 99.187 155.956 0)
+		(effects
+			(font
+				(size 1.27 1.27)
+				(color 255 153 0 1)
+			)
+			(justify left bottom)
+		)
+	)
+	(text "Program"
+		(exclude_from_sim no)
+		(at 60.2375 161.2105 0)
+		(effects
+			(font
+				(size 1.27 1.27)
+				(color 255 153 0 1)
+			)
+			(justify right bottom)
+		)
+	)
+	(text "DMX512\n"
+		(exclude_from_sim no)
+		(at 60.2375 163.7505 0)
+		(effects
+			(font
+				(size 1.27 1.27)
+				(color 255 153 0 1)
+			)
+			(justify right bottom)
+		)
+	)
+	(text "I2C USB-PD Phy\n"
+		(exclude_from_sim no)
+		(at 99.695 163.195 0)
+		(effects
+			(font
+				(size 1.27 1.27)
+				(color 255 153 0 1)
+			)
+			(justify left bottom)
+		)
+	)
 	(junction
 		(at 266.7 151.13)
@@
 		)
 	)
-	(text "External IO\n"
-		(exclude_from_sim no)
-		(at 144.78 168.91 0)
-		(effects
-			(font
-				(size 1.27 1.27)
-				(color 255 153 0 1)
-			)
-			(justify left bottom)
-		)
-	)
-	(text "SK6812\n"
-		(exclude_from_sim no)
-		(at 101.0525 171.5295 0)
-		(effects
-			(font
-				(size 1.27 1.27)
-				(color 255 153 0 1)
-			)
-			(justify left bottom)
-		)
-	)
-	(text "PWM Fan Control"
-		(exclude_from_sim no)
-		(at 99.06 158.75 0)
-		(effects
-			(font
-				(size 1.27 1.27)
-				(color 255 153 0 1)
-			)
-			(justify left bottom)
-		)
-	)
-	(text "PWM Valve Control"
-		(exclude_from_sim no)
-		(at 102.87 151.13 0)
-		(effects
-			(font
-				(size 1.27 1.27)
-				(color 255 153 0 1)
-			)
-			(justify left bottom)
-		)
-	)
-	(text "DMX512\n"
-		(exclude_from_sim no)
-		(at 105.9575 176.4505 0)
-		(effects
-			(font
-				(size 1.27 1.27)
-				(color 255 153 0 1)
-			)
-			(justify left bottom)
-		)
-	)
-	(text "PWM Heater"
-		(exclude_from_sim no)
-		(at 101.6 153.67 0)
-		(effects
-			(font
-				(size 1.27 1.27)
-				(color 255 153 0 1)
-			)
-			(justify left bottom)
-		)
-	)
-	(text "Temperature Sensor\n"
-		(exclude_from_sim no)
-		(at 99.187 155.956 0)
-		(effects
-			(font
-				(size 1.27 1.27)
-				(color 255 153 0 1)
-			)
-			(justify left bottom)
-		)
-	)
-	(text "Program"
-		(exclude_from_sim no)
-		(at 60.2375 161.2105 0)
-		(effects
-			(font
-				(size 1.27 1.27)
-				(color 255 153 0 1)
-			)
-			(justify right bottom)
-		)
-	)
-	(text "DMX512\n"
-		(exclude_from_sim no)
-		(at 60.2375 163.7505 0)
-		(effects
-			(font
-				(size 1.27 1.27)
-				(color 255 153 0 1)
-			)
-			(justify right bottom)
-		)
-	)
-	(text "I2C USB-PD Phy\n"
-		(exclude_from_sim no)
-		(at 99.695 163.195 0)
-		(effects
-			(font
-				(size 1.27 1.27)
-				(color 255 153 0 1)
-			)
-			(justify left bottom)
-		)
-	)
 	(global_label "USB_D-"
 		(shape input)
@@
 		(on_board yes)
 		(dnp no)
-		(property "Reference" "R27"
+		(property "Reference" "R14"
 			(at 261.8486 146.1516 0)
 			(effects
@@
 		(on_board yes)
 		(dnp no)
-		(property "Reference" "R26"
+		(property "Reference" "R11"
 			(at 221.2086 143.6116 0)
 			(effects
@@
 		(on_board yes)
 		(dnp no)
-		(property "Reference" "#PWR0168"
+		(property "Reference" "#PWR06"
 			(at 199.39 161.29 0)
 			(effects
@@
 		(on_board yes)
 		(dnp no)
-		(property "Reference" "R26"
+		(property "Reference" "R6"
 			(at 200.8886 143.6116 0)
 			(effects
@@
 		(on_board yes)
 		(dnp no)
-		(property "Reference" "R26"
+		(property "Reference" "R10"
 			(at 211.0486 143.6116 0)
 			(effects
@@
 		(on_board yes)
 		(dnp no)
-		(property "Reference" "R27"
+		(property "Reference" "R15"
 			(at 268.1986 146.1516 0)
 			(effects
@@
 		(on_board yes)
 		(dnp no)
-		(property "Reference" "#PWR0169"
+		(property "Reference" "#PWR026"
 			(at 256.54 146.05 0)
 			(effects
@@
 		(on_board yes)
 		(dnp no)
-		(property "Reference" "D4"
+		(property "Reference" "D3"
 			(at 212.5472 150.1394 90)
 			(effects
@@
 		(on_board yes)
 		(dnp no)
-		(property "Reference" "#PWR0168"
+		(property "Reference" "#PWR016"
 			(at 219.71 161.29 0)
 			(effects
@@
 		(on_board yes)
 		(dnp no)
-		(property "Reference" "D4"
+		(property "Reference" "D1"
 			(at 202.3872 150.1394 90)
 			(effects
@@
 		(on_board yes)
 		(dnp no)
-		(property "Reference" "#PWR0169"
+		(property "Reference" "#PWR015"
 			(at 219.71 146.05 0)
 			(effects
@@
 		(on_board yes)
 		(dnp no)
-		(property "Reference" "#PWR0168"
+		(property "Reference" "#PWR012"
 			(at 209.55 161.29 0)
 			(effects
@@
 		(at 82.55 26.67)
 		(size 22.86 52.07)
+		(exclude_from_sim no)
+		(in_bom yes)
+		(on_board yes)
+		(dnp no)
 		(fields_autoplaced yes)
 		(stroke
@@
 		(at 27.94 26.67)
 		(size 22.86 50.8)
+		(exclude_from_sim no)
+		(in_bom yes)
+		(on_board yes)
+		(dnp no)
 		(fields_autoplaced yes)
 		(stroke
@@
 		)
 	)
+	(embedded_fonts no)
 )
