File: froggy_hw/out.kicad_sch (KiCad schematic)
At the start: 77 parts, among them J13 NTC, J14 VALVE, J15 NOZZLE, J16 FAN, J17 FAN, J18 LED, Q10 AON6262E, Q11 AON6262E, Q12 AO3400A, Q13 AO3400A, Q14 AO3401A, Q15 AO3401A, Q16 AO3400A, Q17 AO3400A, Q4 S8050, Q5 S8050, Q6 S8050, Q7 S8550, Q8 S8050, Q9 S8550

Commit message: moved to esp32
Parts:
- removed C28, C41, C43, C47, C49, C52: 100n, otter:C_0402, symbol Device:C_Small
- removed D11, D13, D16, D7, D9: SK6805-SIDE-G, otter:SK6805-SIDE-G, symbol otter:SK6805-SIDE-G
- removed J17: FAN, Connector_Molex:Molex_KK-254_AE-6410-04A_1x04_P2.54mm_Vertical, symbol Connector_Generic:Conn_01x04
- removed Q12, Q17: AO3400A, Package_TO_SOT_SMD:SOT-23, symbol Transistor_FET:AO3400A
- removed Q15: AO3401A, Package_TO_SOT_SMD:SOT-23, symbol Transistor_FET:AO3401A
- removed Q4, Q5, Q6, Q8: S8050, Package_TO_SOT_SMD:SOT-23, symbol Transistor_BJT:BC817
- removed Q7, Q9: S8550, Package_TO_SOT_SMD:SOT-23, symbol Transistor_BJT:BC807
- removed R10 (x7), R26 (x2): 5k1, otter:R_0402, symbol Device:R_Small
- removed R10: 22k, otter:R_0402, symbol Device:R_Small
- removed R31, R32: 0, otter:R_0402, symbol Device:R_Small
- removed R37, R38, R39, R40: 200, otter:R_0402, symbol Device:R_Small
- removed R41, R42: 20, otter:R_0603, symbol Device:R_Small
- added C2, C4: 4u7, otter:C_0805, symbol Device:C_Small
- added C3, C5: 100n, otter:C_0402, symbol Device:C_Small
- added U2, U3: MIC4416YM4, Package_TO_SOT_SMD:SOT-143, symbol otter:MIC4416
- C39, C40: footprint Capacitor_THT:CP_Radial_D12.5mm_P7.50mm -> Capacitor_THT:CP_Radial_D6.3mm_P2.50mm
- R10: value 100k -> 5k1
- R45: footprint otter:R_0402 -> otter:R_0805
- R46: footprint otter:R_0603 -> otter:R_0805
Connections:
- net +12V is gone; now on net +24V: C39.1, D18.1 (K), J14.1 (Pin_1), Q14.2 (S), R10.2
- net LED_1 is gone; now on net LED_0: Q13.2 (S), R26.2
- net +5V: now also C2.2, C3.2, C4.2, C5.2, U2.3 (VS), U3.3 (VS)
- net GND: now also C2.1, C3.1, C4.1, C5.1, U2.1 (GND), U3.1 (GND)
- net NOZZLE: now also U2.4 (CTL)
- net VALVE: now also U3.4 (CTL)
- net at R46.1: now also U2.2 (GATE)
- net at J18.2 (Pin_2): now also D15.1 (DOUT)
- net at R45.1: now also U3.2 (GATE)
- no-connect marks 3 -> 1
Other:
- note removed: "OD OUTPUT"
- moved on the sheet: C28, C39, C42, C44, C48, C50, C51, D10, D12, D14, D15, D18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

Commit message: updated to new kicad version
Parts:
- renumbered C28 to C35, C28 to C36, C28 to C37, C28 to C38, C28 to C45, R10 to R43, R10 to R44, R26 to R50, R26 to R52, R10 to R53, R10 to R55
Changed lines of the file:
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@@
 (kicad_sch
-	(version 20231120)
+	(version 20250114)
 	(generator "eeschema")
-	(generator_version "8.0")
+	(generator_version "9.0")
 	(paper "A4")
+	(text "100k\n3950\n"
+		(exclude_from_sim no)
+		(at 125.73 49.53 0)
+		(effects
+			(font
+				(size 1.27 1.27)
+			)
+			(justify left bottom)
+		)
+	)
 	(junction
 		(at 91.44 54.61)
@@
 		)
 	)
-	(text "100k\n3950\n"
-		(exclude_from_sim no)
-		(at 125.73 49.53 0)
-		(effects
-			(font
-				(size 1.27 1.27)
-			)
-			(justify left bottom)
-		)
-	)
 	(hierarchical_label "NOZZLE"
 		(shape input)
 		(at 67.31 166.37 180)
-		(fields_autoplaced yes)
 		(effects
 			(font
@@
 		(shape input)
 		(at 153.67 130.81 180)
-		(fields_autoplaced yes)
 		(effects
 			(font
@@
 		(shape input)
 		(at 199.39 34.29 0)
-		(fields_autoplaced yes)
 		(effects
 			(font
@@
 		(shape input)
 		(at 243.84 39.37 0)
-		(fields_autoplaced yes)
 		(effects
 			(font
@@
 		(shape input)
 		(at 88.9 46.99 180)
-		(fields_autoplaced yes)
 		(effects
 			(font
@@
 		(shape input)
 		(at 67.31 106.68 180)
-		(fields_autoplaced yes)
 		(effects
 			(font
@@
 		(on_board yes)
 		(dnp no)
-		(property "Reference" "R26"
+		(property "Reference" "R50"
 			(at 153.4414 125.8316 0)
 			(effects
@@
 		(on_board yes)
 		(dnp no)
-		(property "Reference" "R10"
+		(property "Reference" "R43"
 			(at 99.06 41.91 0)
 			(effects
@@
 		(dnp no)
 		(fields_autoplaced yes)
-		(property "Reference" "#PWR059"
+		(property "Reference" "#PWR0114"
 			(at 196.85 41.91 0)
 			(effects
@@
 		(dnp no)
 		(fields_autoplaced yes)
-		(property "Reference" "C28"
+		(property "Reference" "C45"
 			(at 225.425 38.0935 0)
 			(effects
@@
 		(dnp no)
 		(fields_autoplaced yes)
-		(property "Reference" "R10"
+		(property "Reference" "R53"
 			(at 231.14 29.21 0)
 			(effects
@@
 		(dnp no)
 		(fields_autoplaced yes)
-		(property "Reference" "#PWR034"
+		(property "Reference" "#PWR095"
 			(at 63.5 54.61 0)
 			(effects
@@
 		(dnp no)
 		(fields_autoplaced yes)
-		(property "Reference" "#PWR034"
+		(property "Reference" "#PWR0130"
 			(at 242.57 52.07 0)
 			(effects
@@
 		(dnp no)
 		(fields_autoplaced yes)
-		(property "Reference" "#PWR034"
+		(property "Reference" "#PWR0107"
 			(at 107.95 173.99 0)
 			(effects
@@
 		(dnp no)
 		(fields_autoplaced yes)
-		(property "Reference" "#PWR034"
+		(property "Reference" "#PWR0102"
 			(at 101.6 99.06 0)
 			(effects
@@
 		(dnp no)
 		(fields_autoplaced yes)
-		(property "Reference" "C28"
+		(property "Reference" "C36"
 			(at 78.105 45.7135 0)
 			(effects
@@
 		(on_board yes)
 		(dnp no)
-		(property "Reference" "R10"
+		(property "Reference" "R44"
 			(at 99.06 49.53 0)
 			(effects
@@
 		(dnp no)
 		(fields_autoplaced yes)
-		(property "Reference" "#PWR034"
+		(property "Reference" "#PWR0126"
 			(at 228.6 52.07 0)
 			(effects
@@
 		(dnp no)
 		(fields_autoplaced yes)
-		(property "Reference" "#PWR034"
+		(property "Reference" "#PWR0103"
 			(at 101.6 158.75 0)
 			(effects
@@
 		(dnp no)
 		(fields_autoplaced yes)
-		(property "Reference" "C28"
+		(property "Reference" "C38"
 			(at 107.95 41.9163 0)
 			(effects
@@
 		(dnp no)
 		(fields_autoplaced yes)
-		(property "Reference" "R10"
+		(property "Reference" "R55"
 			(at 245.11 41.91 0)
 			(effects
@@
 		(dnp no)
 		(fields_autoplaced yes)
-		(property "Reference" "C28"
+		(property "Reference" "C37"
 			(at 88.265 49.5235 0)
 			(effects
@@
 		(dnp no)
 		(fields_autoplaced yes)
-		(property "Reference" "#PWR034"
+		(property "Reference" "#PWR0105"
 			(at 107.95 114.3 0)
 			(effects
@@
 		(dnp no)
 		(fields_autoplaced yes)
-		(property "Reference" "C28"
+		(property "Reference" "C35"
 			(at 67.945 45.7135 0)
 			(effects
@@
 		(on_board yes)
 		(dnp no)
-		(property "Reference" "R26"
+		(property "Reference" "R52"
 			(at 169.1386 125.8316 0)
 			(effects
