File: froggy_hw/power_io.kicad_sch (KiCad schematic)
At the start: 53 parts, among them J10 M4, J11 M4, J12 POWER_OUT, J3 Power_DMX_IO, J4 USB_C, J5 NC3FAAH, J6 NC3MAAH-0, J7 M4, J8 M4, J9 M4, U1 STUSB4500, U10 SY8303AIC, U8 SY8303AIC, U9 SY8303AIC

Commit message: moved to esp32
Parts:
- removed C11 (x2), C28 (x2): 100n, otter:C_0402, symbol Device:C_Small
- removed C13 (x2): 100n, otter:C_0603, symbol Device:C_Small
- removed C14: 100u, Capacitor_THT:CP_Radial_D12.5mm_P7.50mm, symbol Device:C_Polarized
- removed C29 (x6): 4u7, otter:C_0805, symbol Device:C_Small
- removed D6: D210, Diode_SMD:D_SOD-123F, symbol Device:D
- removed J12: POWER_OUT, Connector_PinHeader_2.54mm:PinHeader_1x05_P2.54mm_Horizontal, symbol Connector_Generic:Conn_01x05
- removed J3: Power_DMX_IO, Connector_Phoenix_MC:PhoenixContact_MC_1,5_6-G-3.5_1x06_P3.50mm_Horizontal, symbol Connector:Screw_Terminal_01x06
- removed J4: USB_C, otter:USB-C_Power, symbol Connector:USB_C_Receptacle_PowerOnly_6P
- removed J5: NC3FAAH, Connector_Audio:Jack_XLR_Neutrik_NC3FAAH_Horizontal, symbol Connector_Audio:NC3FAAH
- removed J6: NC3MAAH-0, Connector_Audio:Jack_XLR_Neutrik_NC3MAAH-0_Horizontal, symbol Connector_Audio:NC3MAAH-0
- removed L1: 4u7, Inductor_SMD:L_Taiyo-Yuden_MD-4040, symbol Device:L_Small
- removed L1: 4u7, Inductor_SMD:L_1210_3225Metric, symbol Device:L_Small
- removed R10: 5k1, otter:R_0402, symbol Device:R_Small
- removed R10 (x3): 22k, otter:R_0402, symbol Device:R_Small
- removed R16: 133, otter:R_0805, symbol Device:R_Small
- removed R9 (x2): 100k, otter:R_0402, symbol Device:R_Small
- removed U10, U8: SY8303AIC, Package_TO_SOT_SMD:TSOT-23-8, symbol otter:SY8303AIC
- added C17, C53: 4u7, otter:C_0805, symbol Device:C_Small
- added C6: 100u, Capacitor_THT:CP_Radial_D6.3mm_P2.50mm, symbol Device:C_Polarized
- added C7: 100n, otter:C_0402, symbol Device:C_Small
- added D2: D210, Diode_SMD:D_SMA, symbol Device:D
- added J12, J17: MOUNT, MountingHole:MountingHole_2.2mm_M2_Pad_Via, symbol Connector:Screw_Terminal_01x01
- added J19: HOTEND, otter:froggy_PAD, symbol Connector:Screw_Terminal_01x01
- added J2: POWER, Connector_Phoenix_MC:PhoenixContact_MC_1,5_3-G-3.5_1x03_P3.50mm_Horizontal, symbol Connector_Generic:Conn_01x03
- added J3: DMX CARD, MountingHole:MountingHole_2.2mm_M2_Pad_Via, symbol Connector:Screw_Terminal_01x01
- added J4: USB, otter:USB-C 16Pin, symbol Connector:USB_C_Receptacle_USB2.0_16P
- added J5: POWER_OUT, Connector_PinHeader_2.54mm:PinHeader_1x04_P2.54mm_Horizontal, symbol Connector_Generic:Conn_01x04
- added J6: DMX, Connector_PinHeader_2.54mm:PinHeader_1x05_P2.54mm_Horizontal, symbol Connector_Generic:Conn_01x05
- added R2: 133, otter:R_0805, symbol Device:R_Small
- added U12: USBLC6-4, Package_TO_SOT_SMD:SOT-23-6, symbol otter:otter_USBLC6-4
- added U13: AMS1117-3.3, Package_TO_SOT_SMD:SOT-223-3_TabPin2, symbol Regulator_Linear:AMS1117-3.3
- J10, J11: value M4 -> MOUNT; footprint MountingHole:MountingHole_4.3mm_M4_Pad_Via -> MountingHole:MountingHole_2.2mm_M2_Pad_Via
- J7, J8, J9: value M4 -> HOTEND; footprint MountingHole:MountingHole_4.3mm_M4_Pad_Via -> otter:froggy_PAD
Connections:
- net +24V: now also C6.1, D2.1 (K), J2.2 (Pin_2), J4.A4 (VBUS), J4.A9 (VBUS), J4.B4 (VBUS), J4.B9 (VBUS), J5.2 (Pin_2)
- net +3V3: now also C53.2, J5.4 (Pin_4), U13.2 (VO)
- net +5V: now also C17.2, C7.1, J5.3 (Pin_3), J6.5 (Pin_5), U12.5 (VBUS), U13.3 (VI)
- net GND: now also C17.1, C53.1, C6.2, C7.2, D2.2 (A), J12.1 (Pin_1), J17.1 (Pin_1), J19.1 (Pin_1), J2.1 (Pin_1), J3.1 (Pin_1), J4.A1 (GND), J4.A12 (GND), J4.B1 (GND), J4.B12 (GND), J4.S1 (SHIELD), J5.1 (Pin_1), J6.1 (Pin_1), U12.2 (GND), U13.1 (GND)
- net IO: now also R2.2
- net at U1.1 (CC1DB), U1.2 (CC1): now also J4.A5 (CC1)
- net at U1.4 (CC2), U1.5 (CC2DB): now also J4.B5 (CC2)
- new net: J2.3 (Pin_3), R2.1
- new net RS485_DE: J6.2 (Pin_2)
- new net RS485_RX: J6.3 (Pin_3)
- new net RS485_TX: J6.4 (Pin_4)
- new net USB_D+: J4.A6 (D+), J4.B6 (D+), U12.1 (IO1)
- new net USB_D-: J4.A7 (D-), J4.B7 (D-), U12.3 (IO2)
- no-connect marks 8 -> 12
Other:
- moved on the sheet: C11, C13, C28, C29, L1, R10, R9, U9

Commit message: updated to new kicad version
Parts:
- renumbered C1 to C12, C2 to C13, C3 to C15, C4 to C16, C29 to C18, C11 to C21, C13 to C24, C28 to C27, C29 to C30, C29 to C33, L1 to L3, R3 to R17, R4 to R18, R10 to R23, R9 to R27, R10 to R28, U1 to U7
Changed lines of the file:
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@@
 (kicad_sch
-	(version 20231120)
+	(version 20250114)
 	(generator "eeschema")
-	(generator_version "8.0")
+	(generator_version "9.0")
 	(paper "A4")
+	(text "12V - 28V\n"
+		(exclude_from_sim no)
+		(at 45.72 50.8 0)
+		(effects
+			(font
+				(size 1.27 1.27)
+			)
+			(justify left bottom)
+		)
+	)
 	(junction
 		(at 127 180.34)
@@
 		)
 	)
-	(text "12V - 28V\n"
-		(exclude_from_sim no)
-		(at 45.72 50.8 0)
-		(effects
-			(font
-				(size 1.27 1.27)
-			)
-			(justify left bottom)
-		)
-	)
 	(hierarchical_label "RS485_RX"
 		(shape input)
 		(at 151.13 176.53 0)
-		(fields_autoplaced yes)
 		(effects
 			(font
@@
 		(shape input)
 		(at 109.22 76.2 0)
-		(fields_autoplaced yes)
 		(effects
 			(font
@@
 		(shape input)
 		(at 151.13 179.07 0)
-		(fields_autoplaced yes)
 		(effects
 			(font
@@
 		(shape input)
 		(at 105.41 172.72 0)
-		(fields_autoplaced yes)
 		(effects
 			(font
@@
 		(shape input)
 		(at 109.22 73.66 0)
-		(fields_autoplaced yes)
 		(effects
 			(font
@@
 		(shape input)
 		(at 57.15 104.14 0)
-		(fields_autoplaced yes)
 		(effects
 			(font
@@
 		(shape input)
 		(at 151.13 173.99 0)
-		(fields_autoplaced yes)
 		(effects
 			(font
@@
 		(shape input)
 		(at 55.88 104.14 180)
-		(fields_autoplaced yes)
 		(effects
 			(font
@@
 		(dnp no)
 		(fields_autoplaced yes)
-		(property "Reference" "#PWR034"
+		(property "Reference" "#PWR077"
 			(at 246.38 130.81 0)
 			(effects
@@
 		(on_board yes)
 		(dnp no)
-		(property "Reference" "C3"
+		(property "Reference" "C15"
 			(at 111.5568 38.2016 0)
 			(effects
@@
 		(on_board yes)
 		(dnp no)
-		(property "Reference" "#PWR0112"
+		(property "Reference" "#PWR037"
 			(at 59.69 48.26 0)
 			(effects
@@
 		(dnp no)
 		(fields_autoplaced yes)
-		(property "Reference" "C29"
+		(property "Reference" "C18"
 			(at 185.42 118.1036 0)
 			(effects
@@
 		(on_board yes)
 		(dnp no)
-		(property "Reference" "#PWR0106"
+		(property "Reference" "#PWR045"
 			(at 67.31 87.63 0)
 			(effects
@@
 		(on_board yes)
 		(dnp no)
-		(property "Reference" "#PWR0114"
+		(property "Reference" "#PWR050"
 			(at 109.22 48.26 0)
 			(effects
@@
 		(on_board yes)
 		(dnp no)
-		(property "Reference" "#PWR0107"
+		(property "Reference" "#PWR048"
 			(at 88.9 91.44 0)
 			(effects
@@
 		(dnp no)
 		(fields_autoplaced yes)
-		(property "Reference" "C28"
+		(property "Reference" "C27"
 			(at 243.205 120.6435 0)
 			(effects
@@
 		(on_board yes)
 		(dnp no)
-		(property "Reference" "C4"
+		(property "Reference" "C16"
 			(at 120.4468 38.2016 0)
 			(effects
@@
 		(dnp no)
 		(fields_autoplaced yes)
-		(property "Reference" "#PWR027"
+		(property "Reference" "#PWR080"
 			(at 255.27 130.81 0)
 			(effects
@@
 		(on_board yes)
 		(dnp no)
-		(property "Reference" "#PWR0113"
+		(property "Reference" "#PWR051"
 			(at 114.3 31.75 0)
 			(effects
@@
 		(dnp no)
 		(fields_autoplaced yes)
-		(property "Reference" "L1"
+		(property "Reference" "L3"
 			(at 231.14 113.03 90)
 			(effects
@@
 		(on_board yes)
 		(dnp no)
-		(property "Reference" "#PWR0111"
+		(property "Reference" "#PWR044"
 			(at 67.31 48.26 0)
 			(effects
@@
 		(dnp no)
 		(fields_autoplaced yes)
-		(property "Reference" "C11"
+		(property "Reference" "C21"
 			(at 200.025 118.1035 0)
 			(effects
@@
 		(dnp no)
 		(fields_autoplaced yes)
-		(property "Reference" "R9"
+		(property "Reference" "R27"
 			(at 233.68 120.65 0)
 			(effects
@@
 		(dnp no)
 		(fields_autoplaced yes)
-		(property "Reference" "R3"
+		(property "Reference" "R17"
 			(at 64.77 62.23 90)
 			(effects
@@
 		(dnp no)
 		(fields_autoplaced yes)
-		(property "Reference" "C29"
+		(property "Reference" "C30"
 			(at 252.73 120.6436 0)
 			(effects
@@
 		(dnp no)
 		(fields_autoplaced yes)
-		(property "Reference" "C13"
+		(property "Reference" "C24"
 			(at 222.2436 109.22 90)
 			(effects
@@
 		(dnp no)
 		(fields_autoplaced yes)
-		(property "Reference" "C29"
+		(property "Reference" "C33"
 			(at 261.62 120.6436 0)
 			(effects
@@
 		(dnp no)
 		(fields_autoplaced yes)
-		(property "Reference" "#PWR060"
+		(property "Reference" "#PWR039"
 			(at 60.96 171.45 0)
 			(effects
@@
 		(dnp no)
 		(fields_autoplaced yes)
-		(property "Reference" "#PWR022"
+		(property "Reference" "#PWR065"
 			(at 196.85 128.27 0)
 			(effects
@@
 		(dnp no)
 		(fields_autoplaced yes)
-		(property "Reference" "R10"
+		(property "Reference" "R28"
 			(at 238.76 128.27 0)
 			(effects
@@
 		(on_board yes)
 		(dnp no)
-		(property "Reference" "#PWR0115"
+		(property "Reference" "#PWR052"
 			(at 118.11 48.26 0)
 			(effects
@@
 		(on_board yes)
 		(dnp no)
-		(property "Reference" "U1"
+		(property "Reference" "U7"
 			(at 99.06 83.82 0)
 			(effects
@@
 		(on_board yes)
 		(dnp no)
-		(property "Reference" "C1"
+		(property "Reference" "C12"
 			(at 60.96 36.83 0)
 			(effects
@@
 		(dnp no)
 		(fields_autoplaced yes)
-		(property "Reference" "#PWR053"
+		(property "Reference" "#PWR085"
 			(at 264.16 130.81 0)
 			(effects
@@
 		(dnp no)
 		(fields_autoplaced yes)
-		(property "Reference" "#PWR023"
+		(property "Reference" "#PWR061"
 			(at 187.96 128.27 0)
 			(effects
@@
 		(on_board yes)
 		(dnp no)
-		(property "Reference" "C2"
+		(property "Reference" "C13"
 			(at 68.58 36.83 0)
 			(effects
@@
 		(dnp no)
 		(fields_autoplaced yes)
-		(property "Reference" "#PWR059"
+		(property "Reference" "#PWR071"
 			(at 218.44 134.62 0)
 			(effects
@@
 		(on_board yes)
 		(dnp no)
-		(property "Reference" "R4"
+		(property "Reference" "R18"
 			(at 113.03 83.9216 90)
 			(effects
@@
 		(dnp no)
 		(fields_autoplaced yes)
-		(property "Reference" "R10"
+		(property "Reference" "R23"
 			(at 220.98 124.46 0)
 			(effects
@@
 		(dnp no)
 		(fields_autoplaced yes)
-		(property "Reference" "#PWR059"
+		(property "Reference" "#PWR074"
 			(at 236.22 138.43 0)
 			(effects
@@
 		(dnp no)
 		(fields_autoplaced yes)
-		(property "Reference" "#PWR021"
+		(property "Reference" "#PWR068"
 			(at 205.74 129.54 0)
 			(effects
@@
 		(on_board yes)
 		(dnp no)
-		(property "Reference" "#PWR0108"
+		(property "Reference" "#PWR053"
 			(at 118.11 88.9 0)
 			(effects
